File: Embedded/Synth Head GPU/_autosave-Synth Head GPU.kicad_sch (KiCad schematic)
At the start: 25 parts, among them J1 10171746-00021LF, U11 SRV05-4

Commit message: Added Power and USBC to GPU
Parts:
- removed R11, R12: R, symbol Device:R
Connections:
- net 3V3 Regulator/Vin renamed 1V8 Regulator/Vin
Other:
- sheet 1V8 Regulator ports: added 1V8, Vin; removed none
