File: Embedded/Synth Head GPU/Synth Head GPU.kicad_sch (KiCad schematic)
At the start: 31 parts, among them J1 10171746-00021LF, J2 JST [D], J3 JST [D], J4 JST [G], U10 FFC [G], U11 SRV05-4, U13 TCA9535RTWR, U5 FFC [D], U6 FFC [D], U7 FFC [C], U8 FFC [C], U9 FFC [U]

Commit message: Test Update
Connections:
- net 1V8 Regulator/Vin is gone; now on net +5V: C12.1, J1.A4_B9 (VBUS_A), J1.B4_A9 (VBUS_B)
Changed lines of the file:
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@@
+	)
+	(symbol
+		(lib_id "power:+5V")
+		(at 66.04 74.93 0)
+		(unit 1)
+		(exclude_from_sim no)
+		(in_bom yes)
+		(on_board yes)
+		(dnp no)
+		(fields_autoplaced yes)
+		(property "Reference" "#PWR090"
+			(at 66.04 78.74 0)
+			(effects
+				(font
+					(size 1.27 1.27)
+				)
+				(hide yes)
+			)
+		)
+		(property "Value" "+5V"
+			(at 66.04 69.85 0)
+			(effects
+				(font
+					(size 1.27 1.27)
+				)
+			)
+		)
+		(property "Footprint" ""
+			(at 66.04 74.93 0)
+			(effects
+				(font
+					(size 1.27 1.27)
+				)
+				(hide yes)
+			)
+		)
+		(property "Datasheet" ""
+			(at 66.04 74.93 0)
+			(effects
+				(font
+					(size 1.27 1.27)
+				)
+				(hide yes)
+			)
+		)
+		(property "Description" "Power symbol creates a global label with name \"+5V\""
+			(at 66.04 74.93 0)
+			(effects
+				(font
+					(size 1.27 1.27)
+				)
+				(hide yes)
+			)
+		)
+		(pin "1"
+		)
+		(instances
+			(project ""
+				(path "/4998c09e-38fe-44d6-8b9c-0225a8617744"
+					(reference "#PWR090")
+					(unit 1)
+				)
+			)
+		)
 	)
 	(symbol
