File: Embedded/Synth Head BMS/Synth Head BMS.kicad_sch (KiCad schematic)
At the start: 0 parts

Commit message: PDU Nearly Complete
Parts:
- added J1: JST [P], symbol Connector:Conn_01x12_Socket
Connections:
- new net GND: J1.1 (Pin_1), J1.10 (Pin_10), J1.11 (Pin_11), J1.12 (Pin_12), J1.2 (Pin_2), J1.3 (Pin_3)
- new net Raw PWR: J1.4 (Pin_4), J1.5 (Pin_5), J1.6 (Pin_6), J1.7 (Pin_7), J1.8 (Pin_8), J1.9 (Pin_9)
