File: Embedded/Synth Head CPU/Synth Head CPU.kicad_pcb (KiCad board)
At the start: 2 copper layers, 60 x 35 mm, 56 parts, among them J1 10171746-00021LF, J2 JST [C], J3 MSD-1-A, J4 JST [N], J5 U.FL-R-SMT-1_10_, J6 Pogo JST, J7 Pogo JST, Q1 BSS138, Q2 BSS138, U1 ICM-20948, U2 BME280, U3 AP7366-33W5-7, U4 AP7366-W5-7, U5 FFC [G], U6 FFC [M], U7 FFC [K], U8 NEO-M8M, U9 SRV05-4

Commit message: Prepared Circuits for Routing and Placement Tuning
Parts:
- removed D2: WL-SMCW_0603, LED_Red_SMD:WL-SMCW_0603
- removed R13: 65, Resistor_SMD:R_0603_1608Metric_Pad0.98x0.95mm_HandSolder
- C16, C17, J3: moved to B.Cu
- moved U8 60.7 mm to (166.5, 100.5), turned to 90 degrees
- moved C4 54.4 mm to (150.5, 94.5)
- moved U2 53.5 mm to (150.6, 97.0)
- moved C5 51.9 mm to (150.5, 99.5)
- moved L2 48.8 mm to (169.0, 110.0)
- moved J4 47.7 mm to (120.7, 87.8), turned to -90 degrees
- moved R11 47.5 mm to (168.5, 108.5), turned to 180 degrees
- moved J5 46.4 mm to (172.5, 109.5)
- moved U7 45.9 mm to (160.5, 90.8), turned to 180 degrees
- moved C6 45.4 mm to (120.9, 113.0)
- moved C12 45.1 mm to (156.5, 109.5), turned to 90 degrees
- moved C1 44.7 mm to (154.6, 94.5), turned to 180 degrees
- moved C2 44.3 mm to (157.3, 97.5), turned to 90 degrees
- moved C10 44.3 mm to (152.0, 106.5)
- moved C3 43.7 mm to (154.8, 100.5), turned to 180 degrees
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Connections:
- net CPU-PDU Analog Current renamed CPU-PDU SCL
- net CPU-PDU Analog Voltage renamed CPU-PDU SDA
- U7 pad 3: +5V -> USB +
- U7 pad 4: +5V -> USB -

Commit message: CPU PCB Done
Parts:
- moved R7 1.51 mm to (146.5, 99.9)
- moved R8 1.49 mm to (148.0, 99.9)
- moved U4 1.23 mm to (153.9, 115.0)
- moved C13 1.23 mm to (153.4, 112.3)
- moved C14 1.23 mm to (156.4, 114.8)
- moved C15 1.23 mm to (157.9, 114.8)
- moved R5 1.23 mm to (153.9, 117.8)
- moved R6 1.23 mm to (151.4, 116.8)
- moved C1 0.64 mm to (154.0, 94.5), turned to 0 degrees
- moved R11 0.30 mm to (168.2, 108.5)
- moved BootSW1 0.10 mm to (144.2, 95.9)
- moved L2 0.10 mm to (168.9, 110.0)
- moved R2 0.10 mm to (143.2, 93.4)
Connections:
- ESP1 pad 10: unconnected-(ESP1-GPIO17/U1TXD/ADC2_CH6-Pad10) -> GPS Reset
- ESP1 pad 11: unconnected-(ESP1-GPIO18/U1RXD/ADC2_CH7/CLK_OUT3-Pad11) -> 3V3 Jaw LEDS
- ESP1 pad 17: unconnected-(ESP1-GPIO9/TOUCH9/ADC1_CH8/FSPIHD/SUBSPIHD-Pad17) -> GPS UART TX
- ESP1 pad 18: unconnected-(ESP1-GPIO10/TOUCH10/ADC1_CH9/FSPICS0/FSPIIO4/SUBSPICS0-Pad18) -> GPS UART RX
- ESP1 pad 19: unconnected-(ESP1-GPIO11/TOUCH11/ADC2_CH0/FSPID/FSPIIO5/SUBSPID-Pad19) -> SDA
- ESP1 pad 20: unconnected-(ESP1-GPIO12/TOUCH12/ADC2_CH1/FSPICLK/FSPIIO6/SUBSPICLK-Pad20) -> SCL
- ESP1 pad 21: unconnected-(ESP1-GPIO13/TOUCH13/ADC2_CH2/FSPIQ/FSPIIO7/SUBSPIQ-Pad21) -> CPU-PDU SCL
- ESP1 pad 22: unconnected-(ESP1-GPIO14/TOUCH14/ADC2_CH3/FSPIWP/FSPIDQS/SUBSPIWP-Pad22) -> CPU-PDU SDA
- ESP1 pad 23: unconnected-(ESP1-GPIO21-Pad23) -> CPU-Mask RX
- ESP1 pad 24: unconnected-(ESP1-GPIO47/SPICLK_P/SUBSPICLK_P_DIFF-Pad24) -> CPU-Mask TX
- ESP1 pad 28: unconnected-(ESP1-SPIIO6/GPIO35/FSPID/SUBSPID-Pad28) -> CPU-GPU GPIO 2
- ESP1 pad 29: unconnected-(ESP1-SPIIO7/GPIO36/FSPICLK/SUBSPICLK-Pad29) -> CPU-GPU GPIO 3
- ESP1 pad 30: unconnected-(ESP1-SPIDQS/GPIO37/FSPIQ/SUBSPIQ-Pad30) -> CPU-GPU TX
- ESP1 pad 31: unconnected-(ESP1-GPIO38/FSPIWP/SUBSPIWP-Pad31) -> CPU-GPU RX
- ESP1 pad 32: unconnected-(ESP1-MTCK/GPIO39/CLK_OUT3/SUBSPICS1-Pad32) -> CPU-GPU GPIO 1
- ESP1 pad 33: unconnected-(ESP1-MTDO/GPIO40/CLK_OUT2-Pad33) -> CPU-GPU GPIO 0
- ESP1 pad 34: unconnected-(ESP1-MTDI/GPIO41/CLK_OUT1-Pad34) -> CPU-Mask GPIO 1
- ESP1 pad 35: unconnected-(ESP1-MTMS/GPIO42-Pad35) -> CPU-Mask GPIO 0
- ESP1 pad 4: unconnected-(ESP1-GPIO4/TOUCH4/ADC1_CH3-Pad4) -> 3V3 Neck LEDS
- ESP1 pad 5: unconnected-(ESP1-GPIO5/TOUCH5/ADC1_CH4-Pad5) -> SD Card CS
- ESP1 pad 6: unconnected-(ESP1-GPIO6/TOUCH6/ADC1_CH5-Pad6) -> SD Card MOSI
- ESP1 pad 7: unconnected-(ESP1-GPIO7/TOUCH7/ADC1_CH6-Pad7) -> SD Card CLK
- ESP1 pad 8: unconnected-(ESP1-GPIO15/U0RTS/ADC2_CH4/XTAL_32K_P-Pad8) -> SD Card MISO
- ESP1 pad 9: unconnected-(ESP1-GPIO16/U0CTS/ADC2_CH5/XTAL_32K_N-Pad9) -> SD Card Detect
Routing:
- net +5V: track 0.00 -> 148.4 mm, vias 0 -> 7
- net +3V3: track 0.00 -> 131.5 mm, vias 0 -> 19
- net GPS Reset: track 0.00 -> 59.9 mm, vias 0 -> 2
- net USB -: track 0.00 -> 53.2 mm, vias 0 -> 4
- net USB +: track 0.00 -> 51.9 mm, vias 0 -> 4
- net GND: track 0.00 -> 45.0 mm, vias 0 -> 46
- net +1V8: track 0.00 -> 39.5 mm, vias 0 -> 2
- net SCL: track 0.00 -> 35.3 mm
- net SDA: track 0.00 -> 33.2 mm, vias 0 -> 2
- net CPU-Mask GPIO 0: track 0.00 -> 30.9 mm
- net 3V3 Neck LEDS: track 0.00 -> 30.8 mm
- net 3V3 Jaw LEDS: track 0.00 -> 29.5 mm, vias 0 -> 4
- net GPS UART TX: track 0.00 -> 28.9 mm
- net CPU-PDU SDA: track 0.00 -> 28.5 mm
- net CPU-Mask GPIO 1: track 0.00 -> 28.0 mm
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- added copper zone on F.Cu, net +3V3
- added copper zone on B.Cu, net GND
