File: Embedded/Synth Head CPU/Synth Head CPU.kicad_sch (KiCad schematic)
At the start: 35 parts, among them J1 10171746-00021LF, J2 JST [C], J3 MSD-1-A, J4 JST [N], J6 Pogo JST, J7 Pogo JST, Q1 BSS138, Q2 BSS138, U5 FFC [G], U6 FFC [M], U7 FFC [K], U9 SRV05-4

Commit message: Prepared Circuits for Routing and Placement Tuning
Parts:
- removed D2: WL-SMCW_0603, LED_Red_SMD:WL-SMCW_0603, symbol LED_Red_SMD:WL-SMCW_0603
- removed R13: 65, Resistor_SMD:R_0603_1608Metric_Pad0.98x0.95mm_HandSolder, symbol Device:R
Changed lines of the file:
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@@
 	)
 	(junction
-		(at 102.87 64.77)
-		(diameter 0)
-		(color 0 0 0 0)
-	)
-	(junction
 		(at 162.56 166.37)
 		(diameter 0)
@@
 	(wire
 		(pts
-			(xy 102.87 64.77) (xy 96.52 64.77)
+			(xy 96.52 64.77) (xy 100.33 64.77)
 		)
 		(stroke
@@
 	(wire
 		(pts
-			(xy 102.87 64.77) (xy 113.03 64.77)
-		)
-		(stroke
-			(width 0)
-			(type default)
-		)
-	)
-	(wire
-		(pts
 			(xy 317.5 200.66) (xy 317.5 203.2)
 		)
@@
 	(symbol
 		(lib_id "Device:R")
-		(at 102.87 76.2 0)
-		(unit 1)
-		(exclude_from_sim no)
-		(in_bom yes)
-		(on_board yes)
-		(dnp no)
-		(fields_autoplaced yes)
-		(property "Reference" "R13"
-			(at 105.41 74.9299 0)
-			(effects
-				(font
-					(size 1.27 1.27)
-				)
-				(justify left)
-			)
-		)
-		(property "Value" "65"
-			(at 105.41 77.4699 0)
-			(effects
-				(font
-					(size 1.27 1.27)
-				)
-				(justify left)
-			)
-		)
-		(property "Footprint" "Resistor_SMD:R_0603_1608Metric_Pad0.98x0.95mm_HandSolder"
-			(at 101.092 76.2 90)
-			(effects
-				(font
-					(size 1.27 1.27)
-				)
-				(hide yes)
-			)
-		)
-		(property "Datasheet" "~"
-			(at 102.87 76.2 0)
-			(effects
-				(font
-					(size 1.27 1.27)
-				)
-				(hide yes)
-			)
-		)
-		(property "Description" "Resistor"
-			(at 102.87 76.2 0)
-			(effects
-				(font
-					(size 1.27 1.27)
-				)
-				(hide yes)
-			)
-		)
-		(pin "2"
-		)
-		(pin "1"
-		)
-		(instances
-			(project "Synth Head CPU"
-				(path "/1910f176-637e-4046-b318-0c2bb78fb766"
-					(reference "R13")
-					(unit 1)
-				)
-			)
-		)
-	)
-	(symbol
-		(lib_id "LED_Red_SMD:WL-SMCW_0603")
-		(at 102.87 69.85 90)
-		(unit 1)
-		(exclude_from_sim no)
-		(in_bom yes)
-		(on_board yes)
-		(dnp no)
-		(fields_autoplaced yes)
-		(property "Reference" "D2"
-			(at 106.68 66.5616 90)
-			(effects
-				(font
-					(size 1.27 1.27)
-				)
-				(justify right)
-			)
-		)
-		(property "Value" "WL-SMCW_0603"
-			(at 106.68 69.1016 90)
-			(effects
-				(font
-					(size 1.27 1.27)
-				)
-				(justify right)
-			)
-		)
-		(property "Footprint" "LED_Red_SMD:WL-SMCW_0603"
-			(at 102.87 69.85 0)
-			(effects
-				(font
-					(size 1.27 1.27)
-				)
-				(justify bottom)
-				(hide yes)
-			)
-		)
-		(property "Datasheet" ""
-			(at 102.87 69.85 0)
-			(effects
-				(font
-					(size 1.27 1.27)
-				)
-				(hide yes)
-			)
-		)
-		(property "Description" ""
-			(at 102.87 69.85 0)
-			(effects
-				(font
-					(size 1.27 1.27)
-				)
-				(hide yes)
-			)
-		)
-		(pin "1"
-		)
-		(pin "2"
-		)
-		(instances
-			(project "Synth Head CPU"
-				(path "/1910f176-637e-4046-b318-0c2bb78fb766"
-					(reference "D2")
-					(unit 1)
-				)
-			)
-		)
-	)
-	(symbol
-		(lib_id "Device:R")
 		(at 162.56 139.7 0)
 		(unit 1)
@@
 	)
 	(symbol
-		(lib_id "power:GND")
-		(at 102.87 80.01 0)
-		(unit 1)
-		(exclude_from_sim no)
-		(in_bom yes)
-		(on_board yes)
-		(dnp no)
-		(fields_autoplaced yes)
-		(property "Reference" "#PWR075"
-			(at 102.87 86.36 0)
-			(effects
-				(font
-					(size 1.27 1.27)
-				)
-				(hide yes)
-			)
-		)
-		(property "Value" "GND"
-			(at 102.87 85.09 0)
-			(effects
-				(font
-					(size 1.27 1.27)
-				)
-			)
-		)
-		(property "Footprint" ""
-			(at 102.87 80.01 0)
-			(effects
-				(font
-					(size 1.27 1.27)
-				)
-				(hide yes)
-			)
-		)
-		(property "Datasheet" ""
-			(at 102.87 80.01 0)
-			(effects
-				(font
-					(size 1.27 1.27)
-				)
-				(hide yes)
-			)
-		)
-		(property "Description" "Power symbol creates a global label with name \"GND\" , ground"
-			(at 102.87 80.01 0)
-			(effects
-				(font
-					(size 1.27 1.27)
-				)
-				(hide yes)
-			)
-		)
-		(pin "1"
-		)
-		(instances
-			(project "Synth Head CPU"
-				(path "/1910f176-637e-4046-b318-0c2bb78fb766"
-					(reference "#PWR075")
-					(unit 1)
-				)
-			)
-		)
-	)
-	(symbol
 		(lib_id "Device:C")
 		(at 312.42 36.83 0)
@@
 	(symbol
 		(lib_id "power:+1V8")
-		(at 113.03 64.77 270)
+		(at 100.33 64.77 270)
 		(unit 1)
 		(exclude_from_sim no)
@@
 		(fields_autoplaced yes)
 		(property "Reference" "#PWR027"
-			(at 109.22 64.77 0)
+			(at 96.52 64.77 0)
 			(effects
 				(font
@@
 		)
 		(property "Value" "+1V8"
-			(at 116.84 64.7699 90)
+			(at 104.14 64.7699 90)
 			(effects
 				(font
@@
 		)
 		(property "Footprint" ""
-			(at 113.03 64.77 0)
+			(at 100.33 64.77 0)
 			(effects
 				(font
@@
 		)
 		(property "Datasheet" ""
-			(at 113.03 64.77 0)
+			(at 100.33 64.77 0)
 			(effects
 				(font
@@
 		)
 		(property "Description" "Power symbol creates a global label with name \"+1V8\""
-			(at 113.03 64.77 0)
+			(at 100.33 64.77 0)
 			(effects
 				(font

Commit message: CPU PCB Done
Connections:
- net 3V3 Jaw LEDS: now also ESP1.11 (GPIO18/U1RXD/ADC2_CH7/CLK_OUT3)
- net 3V3 Neck LEDS: now also ESP1.4 (GPIO4/TOUCH4/ADC1_CH3)
- net CPU-GPU GPIO 0: now also ESP1.33 (MTDO/GPIO40/CLK_OUT2)
- net CPU-GPU GPIO 1: now also ESP1.32 (MTCK/GPIO39/CLK_OUT3/SUBSPICS1)
- net CPU-GPU GPIO 2: now also ESP1.28 (SPIIO6/GPIO35/FSPID/SUBSPID)
- net CPU-GPU GPIO 3: now also ESP1.29 (SPIIO7/GPIO36/FSPICLK/SUBSPICLK)
- net CPU-GPU RX: now also ESP1.31 (GPIO38/FSPIWP/SUBSPIWP)
- net CPU-GPU TX: now also ESP1.30 (SPIDQS/GPIO37/FSPIQ/SUBSPIQ)
- net CPU-Mask GPIO 0: now also ESP1.35 (MTMS/GPIO42)
- net CPU-Mask GPIO 1: now also ESP1.34 (MTDI/GPIO41/CLK_OUT1)
- net CPU-Mask RX: now also ESP1.23 (GPIO21)
- net CPU-Mask TX: now also ESP1.24 (GPIO47/SPICLK_P/SUBSPICLK_P_DIFF)
- net CPU-PDU SCL: now also ESP1.21 (GPIO13/TOUCH13/ADC2_CH2/FSPIQ/FSPIIO7/SUBSPIQ)
- net CPU-PDU SDA: now also ESP1.22 (GPIO14/TOUCH14/ADC2_CH3/FSPIWP/FSPIDQS/SUBSPIWP)
- net GPS Reset: now also ESP1.10 (GPIO17/U1TXD/ADC2_CH6)
- net GPS UART RX: now also ESP1.18 (GPIO10/TOUCH10/ADC1_CH9/FSPICS0/FSPIIO4/SUBSPICS0)
- net GPS UART TX: now also ESP1.17 (GPIO9/TOUCH9/ADC1_CH8/FSPIHD/SUBSPIHD)
- net SCL: now also ESP1.20 (GPIO12/TOUCH12/ADC2_CH1/FSPICLK/FSPIIO6/SUBSPICLK)
- net SD Card CLK: now also ESP1.7 (GPIO7/TOUCH7/ADC1_CH6)
- net SD Card CS: now also ESP1.5 (GPIO5/TOUCH5/ADC1_CH4)
- net SD Card Detect: now also ESP1.9 (GPIO16/U0CTS/ADC2_CH5/XTAL_32K_N)
- net SD Card MISO: now also ESP1.8 (GPIO15/U0RTS/ADC2_CH4/XTAL_32K_P)
- net SD Card MOSI: now also ESP1.6 (GPIO6/TOUCH6/ADC1_CH5)
- net SDA: now also ESP1.19 (GPIO11/TOUCH11/ADC2_CH0/FSPID/FSPIIO5/SUBSPID)
Other:
- moved on the sheet: BootSW1, R2
