File: Embedded/Misc Circuits & Adapters/Misc Circuits & Adapters.kicad_sch (KiCad schematic)
At the start: 17 parts, among them J1 VL53L0X, J10 JST [S], J11 Pogo Pins, J12 Jaw Pogo Cable, J13 To LEDS, J2 JST [D], J3 HUB75 PWR, J4 2.0 IPS Display, J5 I2C OLED, J6 I2C OLED, J7 SPI OLED, J8 SPI OLED, J9 HUB75, U1 FFC [C], U2 FFC [U], U3 FFC [D], U5 FFC [G]

Commit message: Prepared Circuits for Routing and Placement Tuning
Parts:
- J12: footprint (none) -> Connector_PinHeader_2.54mm:PinHeader_1x05_P2.54mm_Vertical
- J13: footprint (none) -> Connector_PinHeader_2.54mm:PinHeader_1x03_P2.54mm_Vertical
- J4: footprint (none) -> Connector_PinHeader_2.54mm:PinHeader_1x08_P2.54mm_Vertical
- J5, J6: footprint (none) -> Connector_PinHeader_2.54mm:PinHeader_1x04_P2.54mm_Vertical
- J7, J8: footprint (none) -> Connector_PinHeader_2.54mm:PinHeader_1x07_P2.54mm_Vertical
- J9: footprint (none) -> Connector_PinHeader_2.54mm:PinHeader_2x08_P2.54mm_Vertical
Connections:
- net +5V: now also J8.6 (Pin_6); no longer J8.7 (Pin_7)
- net GND: now also J8.7 (Pin_7); no longer J8.6 (Pin_6)
Changed lines of the file:
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@@
 	(wire
 		(pts
+			(xy 151.13 96.52) (xy 156.21 96.52)
+		)
+		(stroke
+			(width 0)
+			(type default)
+		)
+	)
+	(wire
+		(pts
 			(xy 101.6 152.4) (xy 106.68 152.4)
 		)
@@
 	(wire
 		(pts
-			(xy 151.13 96.52) (xy 156.21 96.52)
-		)
-		(stroke
-			(width 0)
-			(type default)
-		)
-	)
-	(wire
-		(pts
 			(xy 156.21 45.72) (xy 156.21 40.64)
 		)
@@
 	(wire
 		(pts
-			(xy 153.67 93.98) (xy 151.13 93.98)
-		)
-		(stroke
-			(width 0)
-			(type default)
-		)
-	)
-	(wire
-		(pts
 			(xy 163.83 104.14) (xy 163.83 91.44)
 		)
@@
 	(wire
 		(pts
+			(xy 151.13 93.98) (xy 153.67 93.98)
+		)
+		(stroke
+			(width 0)
+			(type default)
+		)
+	)
+	(wire
+		(pts
 			(xy 151.13 43.18) (xy 153.67 43.18)
 		)
@@
 			)
 		)
-		(property "Footprint" ""
+		(property "Footprint" "Connector_PinHeader_2.54mm:PinHeader_1x04_P2.54mm_Vertical"
 			(at 158.75 35.56 0)
 			(effects
@@
 			)
 		)
-		(property "Footprint" ""
+		(property "Footprint" "Connector_PinHeader_2.54mm:PinHeader_2x08_P2.54mm_Vertical"
 			(at 233.68 54.61 0)
 			(effects
@@
 			)
 		)
-		(property "Footprint" ""
+		(property "Footprint" "Connector_PinHeader_2.54mm:PinHeader_1x04_P2.54mm_Vertical"
 			(at 158.75 60.96 0)
 			(effects
@@
 	(symbol
 		(lib_id "power:GND")
-		(at 151.13 96.52 270)
+		(at 151.13 93.98 270)
 		(unit 1)
 		(exclude_from_sim no)
@@
 		(fields_autoplaced yes)
 		(property "Reference" "#PWR027"
-			(at 144.78 96.52 0)
+			(at 144.78 93.98 0)
 			(effects
 				(font
@@
 		)
 		(property "Value" "GND"
-			(at 147.32 96.5201 90)
+			(at 147.32 93.9801 90)
 			(effects
 				(font
@@
 		)
 		(property "Footprint" ""
-			(at 151.13 96.52 0)
+			(at 151.13 93.98 0)
 			(effects
 				(font
@@
 		)
 		(property "Datasheet" ""
-			(at 151.13 96.52 0)
+			(at 151.13 93.98 0)
 			(effects
 				(font
@@
 		)
 		(property "Description" "Power symbol creates a global label with name \"GND\" , ground"
-			(at 151.13 96.52 0)
+			(at 151.13 93.98 0)
 			(effects
 				(font
@@
 	(symbol
 		(lib_id "power:+5V")
-		(at 151.13 93.98 90)
+		(at 151.13 96.52 90)
 		(unit 1)
 		(exclude_from_sim no)
@@
 		(fields_autoplaced yes)
 		(property "Reference" "#PWR026"
-			(at 154.94 93.98 0)
+			(at 154.94 96.52 0)
 			(effects
 				(font
@@
 		)
 		(property "Value" "+5V"
-			(at 147.32 93.9801 90)
+			(at 147.32 96.5201 90)
 			(effects
 				(font
@@
 		)
 		(property "Footprint" ""
-			(at 151.13 93.98 0)
+			(at 151.13 96.52 0)
 			(effects
 				(font
@@
 		)
 		(property "Datasheet" ""
-			(at 151.13 93.98 0)
+			(at 151.13 96.52 0)
 			(effects
 				(font
@@
 		)
 		(property "Description" "Power symbol creates a global label with name \"+5V\""
-			(at 151.13 93.98 0)
+			(at 151.13 96.52 0)
 			(effects
 				(font
@@
 			)
 		)
-		(property "Footprint" ""
+		(property "Footprint" "Connector_PinHeader_2.54mm:PinHeader_1x07_P2.54mm_Vertical"
 			(at 161.29 86.36 0)
 			(effects
@@
 			)
 		)
-		(property "Footprint" ""
+		(property "Footprint" "Connector_PinHeader_2.54mm:PinHeader_1x05_P2.54mm_Vertical"
 			(at 118.11 147.32 0)
 			(effects
@@
 			)
 		)
-		(property "Footprint" ""
+		(property "Footprint" "Connector_PinHeader_2.54mm:PinHeader_1x03_P2.54mm_Vertical"
 			(at 91.44 149.86 0)
 			(effects
@@
 			)
 		)
-		(property "Footprint" ""
+		(property "Footprint" "Connector_PinHeader_2.54mm:PinHeader_1x08_P2.54mm_Vertical"
 			(at 114.3 50.8 0)
 			(effects
@@
 			)
 		)
-		(property "Footprint" ""
+		(property "Footprint" "Connector_PinHeader_2.54mm:PinHeader_1x07_P2.54mm_Vertical"
 			(at 114.3 78.74 0)
 			(effects
