File: Embedded/Synth Head Mask/Synth Head Mask.kicad_pcb (KiCad board)
At the start: 2 copper layers, 75 x 15 mm, 21 parts, among them J1 JST [S], J2 JST [M], J3 JST [F], J4 JST [F], J5 JST [B], J6 JST [K], J7 Misc Expansion, J8 Misc Expansion, Q1 BSS138, Q2 AS2302, U1 FFC [M], U2 FFC [S], U3 AP7366-33W5-7

Commit message: Prepared Circuits for Routing and Placement Tuning
Parts:
- moved J6 59.2 mm to (170.5, 95.5), turned to -90 degrees
- moved U2 57.5 mm to (179.4, 97.2), turned to 90 degrees
- moved R2 39.8 mm to (161.9, 100.5), turned to -90 degrees
- moved R3 36.3 mm to (155.9, 102.0), turned to 90 degrees
- moved J8 30.7 mm to (131.5, 99.0), turned to 90 degrees
- moved JP3 28.6 mm to (132.0, 95.5)
- moved J2 27.9 mm to (151.9, 92.0), turned to 180 degrees
- moved JP2 27.7 mm to (132.0, 92.5)
- moved Q1 26.1 mm to (164.9, 100.5)
- moved J7 25.4 mm to (131.5, 103.0), turned to 90 degrees
- moved J4 24.2 mm to (149.6, 101.4), turned to -90 degrees
- moved Q2 24.2 mm to (158.8, 102.0)
- moved J5 23.4 mm to (125.0, 99.4), turned to 90 degrees
- moved JP1 22.8 mm to (139.0, 94.3), turned to -90 degrees
- moved J1 21.8 mm to (151.9, 96.5), turned to 180 degrees
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