File: Embedded/Synth Head PDU/Synth Head PDU.kicad_pcb (KiCad board)
At the start: 2 copper layers, 40 x 20 mm, 34 parts, among them J1 10171746-00021LF, J2 JST [P], J3 JST [P], J4 JST [USB], J5 JST [C], J6 JST [B], J7 JST [G], Q1 RQ3E100BNTB, Q2 RQ3E100BNTB, U1 FFC [K], U2 TMCS1108A2BQDR, U3 AP7366-33W5-7, U4 RSC002P03, U5 ADS1015IDGS

Commit message: Prepared Circuits for Routing and Placement Tuning
Parts:
- J1, U1: moved to B.Cu
- J4: footprint Connector_PinHeader_2.54mm:PinHeader_1x06_P2.54mm_Vertical -> Connector_PinHeader_1.27mm:PinHeader_1x06_P1.27mm_Vertical
- J5, J6: footprint Connector_PinHeader_2.54mm:PinHeader_1x04_P2.54mm_Vertical -> Connector_Molex:Molex_PicoBlade_53048-0410_1x04_P1.25mm_Horizontal; moved to B.Cu
- moved VR1 48.1 mm to (161.0, 82.5)
- moved J3 43.4 mm to (168.5, 81.1)
- moved VR2 41.3 mm to (139.0, 82.5)
- moved J5 31.7 mm to (159.6, 112.5)
- moved F1 30.4 mm to (152.1, 95.5), turned to -90 degrees
- moved U3 27.1 mm to (139.3, 100.0), turned to 90 degrees
- moved C2 26.1 mm to (136.5, 100.0), turned to 90 degrees
- moved R5 24.4 mm to (143.5, 94.5), turned to 180 degrees
- moved C4 22.2 mm to (139.8, 102.5), turned to 180 degrees
- moved D1 21.8 mm to (147.5, 99.0), turned to -90 degrees
- moved C3 21.8 mm to (139.5, 97.5), turned to 180 degrees
- moved Q2 20.6 mm to (136.0, 87.0), turned to -90 degrees
- moved R10 20.1 mm to (143.5, 102.0)
- moved R9 16.5 mm to (143.5, 103.5), turned to 180 degrees
- moved U2 14.4 mm to (157.5, 102.5), turned to -90 degrees
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Other:
- board size 40 x 20 mm -> 40 x 35 mm
- board text added: "35mm x 40mm"
- board text removed: "20mm x 40mm"
