File: Embedded/Synth Head Snoot/Synth Head Snoot.kicad_pcb (KiCad board)
At the start: 2 copper layers, 55 x 40 mm, 27 parts, among them J1 JST [A], J2 10171746-00021LF, J3 JST [K], J4 MSD-1-A, J5 Touch Pad, J6 Touch Pad, U1 FFC [S], U2 SRV05-4, U3 AP7366-33W5-7, U4 MAX98357AETE_T

Commit message: Prepared Circuits for Routing and Placement Tuning
Parts:
- C3: footprint Capacitor_SMD:C_0603_1608Metric -> Capacitor_SMD:C_0603_1608Metric_Pad1.08x0.95mm_HandSolder
- J4, J5, TP1: moved to B.Cu
- moved TP2 69.5 mm to (172.5, 90.5)
- moved C7 53.9 mm to (152.5, 103.3)
- moved J6 51.7 mm to (172.5, 85.5)
- moved C6 48.3 mm to (150.0, 106.0), turned to -90 degrees
- moved TP1 47.2 mm to (141.0, 88.5), turned to 180 degrees
- moved C5 46.4 mm to (152.8, 109.0), turned to 180 degrees
- moved U3 46.1 mm to (152.5, 106.0), turned to 180 degrees
- moved R2 45.9 mm to (129.5, 84.3), turned to 90 degrees
- moved J5 44.2 mm to (141.0, 85.5), turned to 180 degrees
- moved BootSW1 38.0 mm to (127.0, 84.5), turned to -90 degrees
- moved R1 34.9 mm to (152.0, 96.0), turned to 180 degrees
- moved C1 29.6 mm to (152.0, 94.5), turned to 180 degrees
- moved JP1 29.5 mm to (135.5, 106.0), turned to 180 degrees
- moved C3 27.8 mm to (151.0, 98.5), turned to -90 degrees
- moved L1 26.6 mm to (149.0, 111.0), turned to 90 degrees
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